File: circuit/SERN.kicad_pcb (KiCad board)
At the start: 2 copper layers, 100 x 100 mm, 71 parts, among them J1 Conn_01x03, J2 Conn_01x04, J3 RaspberryPi3, J4 Conn_01x03, J5 Conn_01x03, U1 MCW03, U2 NE5534, U3 NE5534, U4 ICS570, U5 pcm1794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

Commit message: [add]製造データできた
Other:
- net class Default: clearance 0.2 -> 0.254; trace_width 0.25 -> 0.254
- rule trace_clearance: 0.2 -> 0.254
- rule via_min_drill: 0.3 -> 0.4
- rule via_min_size: 0.4 -> 0.6
- board text added: "SERN PROJECT 2018 Designed in NITTC"
Changed lines of the file:
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@@
     (links 166)
     (no_connects 0)
-    (area 39.949999 39.949999 140.050001 140.050001)
+    (area 34.192857 38.575 145.807143 141.525)
     (thickness 1.6)
-    (drawings 4)
+    (drawings 5)
     (tracks 550)
     (zones 0)
@@
   )
   (setup
-    (last_trace_width 0.25)
+    (last_trace_width 0.254)
     (user_trace_width 3.5)
-    (trace_clearance 0.2)
+    (trace_clearance 0.254)
     (zone_clearance 0.508)
     (zone_45_only no)
@@
     (via_size 0.6)
     (via_drill 0.4)
-    (via_min_size 0.4)
-    (via_min_drill 0.3)
+    (via_min_size 0.6)
+    (via_min_drill 0.4)
     (uvia_size 0.3)
     (uvia_drill 0.1)
@@
       (outputformat 1)
       (mirror false)
-      (drillshape 1)
+      (drillshape 0)
       (scaleselection 1)
-      (outputdirectory ""))
+      (outputdirectory PRODUCTION_FILE/))
   )
   (net 0 "")
@@
   (net 84 GNDD)
   (net_class Default "これは標準のネット クラスです。"
-    (clearance 0.2)
-    (trace_width 0.25)
+    (clearance 0.254)
+    (trace_width 0.254)
     (via_dia 0.6)
     (via_drill 0.4)
@@
     (pad 1 np_thru_hole circle (at 0 0) (size 3.2 3.2) (drill 3.2) (layers *.Cu *.Mask))
   )
+  (gr_text "SERN PROJECT 2018\nDesigned in NITTC" (at 62.5 135) (layer F.SilkS)
+    (effects (font (size 1.5 1.5) (thickness 0.3)))
+  )
   (gr_line (start 140 40) (end 40 40) (angle 90) (layer Edge.Cuts) (width 0.1))
